Commit message: improved tfs

File: panther_gazebo/urdf/quadrotor_with_asus.urdf.xacro (robot description, xacro)
@@ -10,5 +10,5 @@
     <xacro:asus_camera name="camera" parent="base_link">
      <!-- <origin xyz="0.1 0.0 -0.03" rpy="0 0 0"/>-->
-         <origin xyz="0.1 0.0 0" rpy="0 0 0"/>
+         <origin xyz="0.1 0.0 0" rpy="0 0.0 0"/>  <!-- 0 -0.78 0 -->
     </xacro:asus_camera>
        <!-- Sonar height sensor -->
